File: kicad/breakout-board.sch (KiCad schematic (older format))
At the start: 18 parts, among them IC1 ATMEGA328-P, P1 CONN_01X02, P2 Conn_3, P3 Conn_2b, P4 Conn_1, P5 Conn_5, P6 Conn_6, P7 Conn_4, P8 Conn_2b, P9 6Pin Connector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

Commit message: redesign fully header connected
Parts:
- removed P6: Conn_6, Pin_Headers:Pin_Header_Straight_1x04, symbol CONN_01X04
- removed P7: Conn_4, Pin_Headers:Pin_Header_Straight_1x04, symbol CONN_01X04
- removed P8: Conn_2b, Pin_Headers:Pin_Header_Straight_1x02, symbol CONN_01X02
- removed Y1: 16MHz, Crystals:Crystal_HC50-U_Vertical, symbol Crystal
- added P10, P11: CONN_01X01, Pin_Headers:Pin_Header_Straight_1x01, symbol CONN_01X01
- added P6, P8: CONN_01X06, Pin_Headers:Pin_Header_Straight_1x06, symbol CONN_01X06
- added P7: CONN_01X02, Pin_Headers:Pin_Header_Straight_1x02, symbol CONN_01X02
- P2: value Conn_3 -> CONN_01X04
- P3: value Conn_2b -> CONN_01X02
- P4: value Conn_1 -> CONN_01X04
- P5: value Conn_5 -> CONN_01X04
Connections:
- net +5V: now also P5.3 (P3), P8.4 (P4)
- net AREF: now also P8.5 (P5); no longer P5.2 (P2)
- net GND: now also P5.4 (P4), P8.6 (P6)
- net MISO: now also P8.2 (P2)
- net MOSI: now also P8.1 (P1)
- net PB0: now also P4.4 (P4); no longer P2.4 (P4)
- net PB1: now also P7.1 (P1)
- net PB2: now also P7.2 (P2)
- net PC0: now also P6.1 (P1); no longer P5.3 (P3)
- net PC1: now also P6.2 (P2); no longer P5.4 (P4)
- net PC2: now also P6.3 (P3)
- net PC3: now also P6.4 (P4)
- net PC4: now also P6.5 (P5)
- net PC5: now also P6.6 (P6)
- net PD0: now also P2.2 (P2); no longer P4.2 (P2)
- net PD1: now also P2.3 (P3); no longer P4.3 (P3)
- net PD2: now also P2.4 (P4); no longer P4.4 (P4)
- net PD3: now also P5.1 (P1)
- net PD4: now also P5.2 (P2)
- net PD5: now also P4.1 (P1); no longer P2.1 (P1)
- net PD6: now also P4.2 (P2); no longer P2.2 (P2)
- net PD7: now also P4.3 (P3); no longer P2.3 (P3)
- net RESET: now also P2.1 (P1); no longer P4.1 (P1)
- net SCK: now also P8.3 (P3); no longer P5.1 (P1)
- net XTAL1: now also P10.1 (P1)
- net XTAL2: now also P11.1 (P1)
Other:
- moved on the sheet: P1

Commit message: redesign mirror and re-place isp, make it smaller
Parts:
- removed P1: CONN_01X02, Pin_Headers:Pin_Header_Straight_1x02, symbol CONN_01X02
- added P1: CONN_01X01, Pin_Headers:Pin_Header_Straight_1x01, symbol CONN_01X01
Connections:
- net +5V: now also P9.5 (P5), P1.1 (P1); no longer P9.1 (P1)
- net GND: now also P9.1 (P1); no longer P9.5 (P5)
- net MISO: now also P9.6 (P6); no longer P9.2 (P2)
- net RESET: now also P9.2 (P2); no longer P9.6 (P6)
Changed lines of the file:
@@
 L GND #PWR05
 U 1 1 568D6628
+P 7190 1450
+F 0 "#PWR05" H 7190 1200 50  0001 C CNN
+F 1 "GND" V 7193 1216 50  0000 C CNN
+F 2 "" H 7190 1450 50  0000 C CNN
+F 3 "" H 7190 1450 50  0000 C CNN
+	1    7190 1450
+	0    1    1    0
+$EndComp
+$Comp
+L +5V #PWR06
+U 1 1 568D6644
 P 7190 1650
-F 0 "#PWR05" H 7190 1400 50  0001 C CNN
-F 1 "GND" V 7230 1470 50  0000 C CNN
+F 0 "#PWR06" H 7190 1500 50  0001 C CNN
+F 1 "+5V" V 7200 1862 50  0000 C CNN
 F 2 "" H 7190 1650 50  0000 C CNN
 F 3 "" H 7190 1650 50  0000 C CNN
 	1    7190 1650
-	0    1    1    0
-$EndComp
-$Comp
-L +5V #PWR06
-U 1 1 568D6644
-P 7190 1450
-F 0 "#PWR06" H 7190 1300 50  0001 C CNN
-F 1 "+5V" V 7220 1640 50  0000 C CNN
-F 2 "" H 7190 1450 50  0000 C CNN
-F 3 "" H 7190 1450 50  0000 C CNN
-	1    7190 1450
 	0    -1   -1   0
 $EndComp
-Text GLabel 7690 1450 2    60   Input ~ 0
+Text GLabel 7690 1650 2    60   Input ~ 0
 MISO
 Text GLabel 7690 1550 2    60   Input ~ 0
 SCK
-Text GLabel 7690 1650 2    60   Input ~ 0
+Text GLabel 7690 1450 2    60   Input ~ 0
 RESET
 Text GLabel 7180 2210 0    60   Input ~ 0
@@
 PD7
 $Comp
-L GND #PWR09
-U 1 1 568DB8F4
-P 6320 3130
-F 0 "#PWR09" H 6320 2880 50  0001 C CNN
-F 1 "GND" H 6320 2980 50  0000 C CNN
-F 2 "" H 6320 3130 50  0000 C CNN
-F 3 "" H 6320 3130 50  0000 C CNN
-	1    6320 3130
-	-1   0    0    -1
-$EndComp
-$Comp
-L +5V #PWR010
+L +5V #PWR09
 U 1 1 568DB9A8
-P 6320 3030
-F 0 "#PWR010" H 6320 2880 50  0001 C CNN
-F 1 "+5V" H 6320 3170 50  0000 C CNN
-F 2 "" H 6320 3030 50  0000 C CNN
-F 3 "" H 6320 3030 50  0000 C CNN
-	1    6320 3030
+P 6195 3034
+F 0 "#PWR09" H 6195 2884 50  0001 C CNN
+F 1 "+5V" H 6195 3174 50  0000 C CNN
+F 2 "" H 6195 3034 50  0000 C CNN
+F 3 "" H 6195 3034 50  0000 C CNN
+	1    6195 3034
 	-1   0    0    -1
 $EndComp
@@
 Power
 $Comp
-L PWR_FLAG #FLG011
+L PWR_FLAG #FLG010
 U 1 1 568DC3F0
 P 1840 850
-F 0 "#FLG011" H 1840 945 50  0001 C CNN
+F 0 "#FLG010" H 1840 945 50  0001 C CNN
 F 1 "PWR_FLAG" H 1840 1030 50  0000 C CNN
 F 2 "" H 1840 850 50  0000 C CNN
@@
 AREF
 $Comp
-L PWR_FLAG #FLG012
+L PWR_FLAG #FLG011
 U 1 1 568DD7E9
 P 1840 3350
-F 0 "#FLG012" H 1840 3445 50  0001 C CNN
+F 0 "#FLG011" H 1840 3445 50  0001 C CNN
 F 1 "PWR_FLAG" H 1840 3530 50  0000 C CNN
 F 2 "" H 1840 3350 50  0000 C CNN
@@
 	1    2488 4098
 	1    0    0    -1
-$EndComp
-$Comp
-L CONN_01X02 P1
-U 1 1 568DB809
-P 6120 3080
-F 0 "P1" H 6120 3230 50  0000 C CNN
-F 1 "CONN_01X02" V 6220 3080 50  0000 C CNN
-F 2 "Pin_Headers:Pin_Header_Straight_1x02" H 6120 3080 50  0001 C CNN
-F 3 "" H 6120 3080 50  0000 C CNN
-	1    6120 3080
-	-1   0    0    -1
 $EndComp
 Wire Wire Line
@@
 	8800 2590 8800 2810
 $Comp
-L GND #PWR013
+L GND #PWR012
 U 1 1 56902ACD
 P 2188 4098
-F 0 "#PWR013" H 2188 3848 50  0001 C CNN
+F 0 "#PWR012" H 2188 3848 50  0001 C CNN
 F 1 "GND" H 2188 3948 50  0000 C CNN
 F 2 "" H 2188 4098 50  0000 C CNN
@@
 $EndComp
 $Comp
-L GND #PWR014
+L GND #PWR013
 U 1 1 56902B08
 P 2788 4098
-F 0 "#PWR014" H 2788 3848 50  0001 C CNN
+F 0 "#PWR013" H 2788 3848 50  0001 C CNN
 F 1 "GND" H 2788 3948 50  0000 C CNN
 F 2 "" H 2788 4098 50  0000 C CNN
@@
 $EndComp
 $Comp
-L +5V #PWR015
+L +5V #PWR014
 U 1 1 56902D67
 P 814 2046
-F 0 "#PWR015" H 814 1896 50  0001 C CNN
+F 0 "#PWR014" H 814 1896 50  0001 C CNN
 F 1 "+5V" H 814 2186 50  0000 C CNN
 F 2 "" H 814 2046 50  0000 C CNN
@@
 $EndComp
 $Comp
-L +5V #PWR016
+L +5V #PWR015
 U 1 1 56902E04
 P 1414 2046
-F 0 "#PWR016" H 1414 1896 50  0001 C CNN
+F 0 "#PWR015" H 1414 1896 50  0001 C CNN
 F 1 "+5V" H 1414 2186 50  0000 C CNN
 F 2 "" H 1414 2046 50  0000 C CNN
@@
 $EndComp
 $Comp
-L GND #PWR017
+L GND #PWR016
 U 1 1 569038E0
 P 1048 4038
-F 0 "#PWR017" H 1048 3788 50  0001 C CNN
+F 0 "#PWR016" H 1048 3788 50  0001 C CNN
 F 1 "GND" H 1048 3888 50  0000 C CNN
 F 2 "" H 1048 4038 50  0000 C CNN
@@
 $EndComp
 $Comp
-L GND #PWR018
+L GND #PWR017
 U 1 1 56903921
 P 1648 4038
-F 0 "#PWR018" H 1648 3788 50  0001 C CNN
+F 0 "#PWR017" H 1648 3788 50  0001 C CNN
 F 1 "GND" H 1648 3888 50  0000 C CNN
 F 2 "" H 1648 4038 50  0000 C CNN
@@
 PC5
 $Comp
-L +5V #PWR019
+L +5V #PWR018
 U 1 1 56A2218E
 P 5820 1862
-F 0 "#PWR019" H 5820 1712 50  0001 C CNN
+F 0 "#PWR018" H 5820 1712 50  0001 C CNN
 F 1 "+5V" H 5820 2002 50  0000 C CNN
 F 2 "" H 5820 1862 50  0000 C CNN
@@
 $EndComp
 $Comp
-L +5V #PWR020
+L +5V #PWR019
 U 1 1 56A221BC
 P 4987 1653
-F 0 "#PWR020" H 4987 1503 50  0001 C CNN
+F 0 "#PWR019" H 4987 1503 50  0001 C CNN
 F 1 "+5V" H 4987 1793 50  0000 C CNN
 F 2 "" H 4987 1653 50  0000 C CNN
@@
 $EndComp
 $Comp
-L GND #PWR021
+L GND #PWR020
 U 1 1 56A221EA
 P 4987 1753
-F 0 "#PWR021" H 4987 1503 50  0001 C CNN
+F 0 "#PWR020" H 4987 1503 50  0001 C CNN
 F 1 "GND" H 4987 1603 50  0000 C CNN
 F 2 "" H 4987 1753 50  0000 C CNN
@@
 $EndComp
 $Comp
-L GND #PWR022
+L GND #PWR021
 U 1 1 56A22218
 P 5820 1662
-F 0 "#PWR022" H 5820 1412 50  0001 C CNN
+F 0 "#PWR021" H 5820 1412 50  0001 C CNN
 F 1 "GND" H 5820 1512 50  0000 C CNN
 F 2 "" H 5820 1662 50  0000 C CNN
@@
 	1    0    0    -1
 $EndComp
+$Comp
+L CONN_01X01 P1
+U 1 1 56A354F0
+P 6195 3234
+F 0 "P1" H 6189 3134 50  0000 C CNN
+F 1 "CONN_01X01" H 6047 3443 50  0000 C CNN
+F 2 "Pin_Headers:Pin_Header_Straight_1x01" H 6195 3234 50  0001 C CNN
+F 3 "" H 6195 3234 50  0000 C CNN
+	1    6195 3234
+	0    1    1    0
+$EndComp
 $EndSCHEMATC
